File: pcb/flipcontrol.kicad_sch (KiCad schematic)
At the start: 45 parts, among them J1 PJ-202A, J2 DOT_BOARD_1, J3 DOT_BOARD_2, J4 LED_STRIP, J5 DOT_BOARD_3, Q1 UMH3N, Q2 Si2347DS-T1-GE3, Q3 MMBT3904, Q4 Si2347DS-T1-GE3, Q5 MMBT3904, U1 LM2596S-5, U2 AMS1117-3.3, U3 CH340C, U3 ESP32-S3-WROOM-1

Commit message: Start work on Ethernet support in schematic
Parts:
- added C10, C11: 6.8nF, symbol Device:C
- added C12: 22nF, symbol Device:C
- added C13, C14: 10nF, symbol Device:C
- added C15: 4.7uF, symbol Device:C
- added C16, C17, C18, C19, C20, C21: 0.1uF, symbol Device:C
- added C22: 10uF/16V, symbol Device:C_Polarized
- added C23: C_Polarized, symbol Device:C_Polarized
- added J6: RJMG163118101NR, RJMG163118101NR, symbol SamacSys_Parts:RJMG163118101NR
- added L2: HH-1M1608-121JT, symbol Device:L
- added R11, R12, R13, R14: 33R, symbol Device:R
- added R15, R16, R18, R19: 49R9, symbol Device:R
- added R17: 10R, symbol Device:R
- added R20: 12.4k, symbol Device:R
- added R21, R22: 330R, symbol Device:R
- added U5: W5500, Package_QFP:LQFP-48_7x7mm_P0.5mm, symbol Interface_Ethernet:W5500
Connections:
- net +3V3: now also J6.L1 (GREEN_A_1), J6.L4 (GREEN_A_2), L2.1
- net GND: now also C12.2, C13.2, C14.2, C15.2, C16.2, C17.2, C18.2, C19.2, C20.2, C21.2, C22.2, R20.2, U5.14 (AGND), U5.16 (AGND), U5.19 (AGND), U5.29 (GND), U5.3 (AGND), U5.48 (AGND), U5.9 (AGND)
- new net: R14.1, R15.2, U5.1 (TXN)
- new net: J6.R3 (TX-), R14.2
- new net: C11.1, R12.1
- new net: R12.2, R18.1, U5.6 (RXP)
- new net: C15.1, U5.20 (TOCAP)
- new net: R11.1, R19.1, U5.5 (RXN)
- new net: C13.1, J6.R6 (RCT), R18.2, R19.2
- new net: R20.1, U5.10 (EXRES1)
- new net: R13.1, R16.2, U5.2 (TXP)
- new net: C14.1, U5.22 (1V2O)
- new net: J6.L2 (GREEN_K_1), R21.1
- new net: J6.L3 (GREEN_K_2), R22.1
- new net: J6.R1 (TCT), R17.1
- new net: J6.R2 (TX+), R13.2
- new net: C11.2, J6.R4 (RX+)
- new net: C10.1, J6.R5 (RX-)
- new net: C10.2, R11.2
- new net +3.3VA: C12.1, C16.1, C17.1, C18.1, C19.1, C20.1, C21.1, C22.1, L2.2, R15.1, R16.1, R17.2, U5.11 (AVDD), U5.15 (AVDD), U5.17 (AVDD), U5.21 (AVDD), U5.4 (AVDD), U5.8 (AVDD)
- new net ACT_LED: R22.2, U5.27 (ACTLED)
- new net LINK_LED: R21.2, U5.25 (LINKLED)
- no-connect marks 21 -> 29
Other:
- moved on the sheet: C2, C3, C4, C5, C8, D1, D2, J1, J2, J3, J4, J5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

Commit message: Finish adding Ethernet interface
Parts:
- added C24: 0.1uF, symbol Device:C
- added C25, C26: 18pF, symbol Device:C
- added R23: 1M, symbol Device:R
- added R24: 4.7k, symbol Device:R
- added Y1: Crystal_GND24, symbol Device:Crystal_GND24
- C23: value C_Polarized -> 10uF/16v
Connections:
- net +3V3: now also C23.1, U5.28 (VDD), U5.43 (PMODE2), U5.44 (PMODE1), U5.45 (PMODE0), C24.1, R24.1
- net COIL_DRIVE_IN: now also U3.38 (GPIO2/TOUCH2/ADC1_CH1); no longer U3.5 (GPIO5/TOUCH5/ADC1_CH4)
- net COL_ADVANCE_1: now also U3.6 (GPIO6/TOUCH6/ADC1_CH5); no longer U3.12 (GPIO8/TOUCH8/ADC1_CH7/SUBSPICS1)
- net COL_ADVANCE_2: now also U3.22 (GPIO14/TOUCH14/ADC2_CH3/FSPIWP/FSPIDQS/SUBSPIWP); no longer U3.11 (GPIO18/U1RXD/ADC2_CH7/CLK_OUT3)
- net COL_ADVANCE_3: now also U3.31 (GPIO38/FSPIWP/SUBSPIWP); no longer U3.16 (GPIO46)
- net ENABLE_1: now also U3.12 (GPIO8/TOUCH8/ADC1_CH7/SUBSPICS1); no longer U3.18 (GPIO10/TOUCH10/ADC1_CH9/FSPICS0/FSPIIO4/SUBSPICS0)
- net ENABLE_2: now also U3.17 (GPIO9/TOUCH9/ADC1_CH8/FSPIHD/SUBSPIHD); no longer U3.19 (GPIO11/TOUCH11/ADC2_CH0/FSPID/FSPIIO5/SUBSPID)
- net ENABLE_3: now also U3.18 (GPIO10/TOUCH10/ADC1_CH9/FSPICS0/FSPIIO4/SUBSPICS0); no longer U3.20 (GPIO12/TOUCH12/ADC2_CH1/FSPICLK/FSPIIO6/SUBSPICLK)
- net ENABLE_4: now also U3.19 (GPIO11/TOUCH11/ADC2_CH0/FSPID/FSPIIO5/SUBSPID); no longer U3.21 (GPIO13/TOUCH13/ADC2_CH2/FSPIQ/FSPIIO7/SUBSPIQ)
- net GND: now also C23.2, C24.2, C25.2, C26.2, Y1.2, Y1.4
- net LED_IN: now also U3.39 (GPIO1/TOUCH1/ADC1_CH0); no longer U3.4 (GPIO4/TOUCH4/ADC1_CH3)
- net RESET_1: now also U3.7 (GPIO7/TOUCH7/ADC1_CH6); no longer U3.17 (GPIO9/TOUCH9/ADC1_CH8/FSPIHD/SUBSPIHD)
- net RESET_2: now also U3.10 (GPIO17/U1TXD/ADC2_CH6); no longer U3.23 (GPIO21)
- net ROW_ADVANCE_1: now also U3.5 (GPIO5/TOUCH5/ADC1_CH4); no longer U3.7 (GPIO7/TOUCH7/ADC1_CH6)
- net ROW_ADVANCE_2: now also U3.21 (GPIO13/TOUCH13/ADC2_CH2/FSPIQ/FSPIIO7/SUBSPIQ); no longer U3.10 (GPIO17/U1TXD/ADC2_CH6)
- net ROW_ADVANCE_3: now also U3.23 (GPIO21); no longer U3.26 (GPIO45)
- net SET_UNSET_1: now also U3.4 (GPIO4/TOUCH4/ADC1_CH3); no longer U3.6 (GPIO6/TOUCH6/ADC1_CH5)
- net SET_UNSET_2: now also U3.20 (GPIO12/TOUCH12/ADC2_CH1/FSPICLK/FSPIIO6/SUBSPICLK); no longer U3.22 (GPIO14/TOUCH14/ADC2_CH3/FSPIWP/FSPIDQS/SUBSPIWP)
- net SET_UNSET_3: now also U3.11 (GPIO18/U1RXD/ADC2_CH7/CLK_OUT3); no longer U3.31 (GPIO38/FSPIWP/SUBSPIWP)
- net MOSI: now reaches U3.28 (SPIIO6/GPIO35/FSPID/SUBSPID)
- net MOSI: now also U5.35 (MOSI)
- net SCLK: now reaches U3.29 (SPIIO7/GPIO36/FSPICLK/SUBSPICLK)
- net SCLK: now also U5.33 (SCLK)
- net MISO: now reaches U3.30 (SPIDQS/GPIO37/FSPIQ/SUBSPIQ)
- net MISO: now also U5.34 (MISO)
- net ETH_RST: now reaches U3.34 (MTDI/GPIO41/CLK_OUT1)
- net ETH_RST: now also U5.37 (~{RST})
- net CS: now reaches U3.35 (MTMS/GPIO42)
- net CS: now also U5.32 (~{SCS})
- net at U5.30 (XI/CLKIN): now also C26.1, R23.2, Y1.1
- net at U5.31 (XO): now also C25.1, R23.1, Y1.3
- net at U5.36 (~{INT}): now also R24.2
- no-connect marks 29 -> 24

Commit message: Add footprints for all parts
Parts:
- C10, C11, C12, C13, C14, C15, C16, C17, C18, C19, C20, C21, C22, C23, C24, C25, C26: footprint (none) -> Capacitor_SMD:C_0805_2012Metric
- J6: footprint RJMG163118101NR -> SamacSys_Parts:RJMG163118101NR
- L2: footprint (none) -> Inductor_SMD:L_0805_2012Metric
- Q2, Q4: footprint SOT95P237X112-3N -> SamacSys_Parts:SOT95P237X112-3N
- R11, R12, R13, R14, R15, R16, R17, R18, R19, R20, R21, R22, R23, R24: footprint (none) -> Resistor_SMD:R_0805_2012Metric
- Y1: footprint (none) -> Crystal:Crystal_SMD_Abracon_ABM8G-4Pin_3.2x2.5mm
Changed lines of the file:
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@@
       (effects (font (size 1.27 1.27)))
     )
-    (property "Footprint" "" (at 341.63 318.008 90)
+    (property "Footprint" "Resistor_SMD:R_0805_2012Metric" (at 341.63 318.008 90)
       (effects (font (size 1.27 1.27)) hide)
     )
@@
       (effects (font (size 1.27 1.27)))
     )
-    (property "Footprint" "" (at 341.63 333.502 90)
+    (property "Footprint" "Resistor_SMD:R_0805_2012Metric" (at 341.63 333.502 90)
       (effects (font (size 1.27 1.27)) hide)
     )
@@
       (effects (font (size 1.27 1.27)))
     )
-    (property "Footprint" "" (at 199.39 360.68 0)
+    (property "Footprint" "Crystal:Crystal_SMD_Abracon_ABM8G-4Pin_3.2x2.5mm" (at 199.39 360.68 0)
       (effects (font (size 1.27 1.27)) hide)
     )
@@
       (effects (font (size 1.27 1.27)) (justify left))
     )
-    (property "Footprint" "" (at 295.6052 306.07 0)
+    (property "Footprint" "Capacitor_SMD:C_0805_2012Metric" (at 295.6052 306.07 0)
       (effects (font (size 1.27 1.27)) hide)
     )
@@
       (effects (font (size 1.27 1.27)))
     )
-    (property "Footprint" "" (at 271.78 369.8748 0)
+    (property "Footprint" "Capacitor_SMD:C_0805_2012Metric" (at 271.78 369.8748 0)
       (effects (font (size 1.27 1.27)) hide)
     )
@@
       (effects (font (size 1.27 1.27)) (justify left))
     )
-    (property "Footprint" "" (at 207.9752 313.69 0)
+    (property "Footprint" "Capacitor_SMD:C_0805_2012Metric" (at 207.9752 313.69 0)
       (effects (font (size 1.27 1.27)) hide)
     )
@@
       (effects (font (size 1.27 1.27)))
     )
-    (property "Footprint" "" (at 436.88 324.1548 0)
+    (property "Footprint" "Capacitor_SMD:C_0805_2012Metric" (at 436.88 324.1548 0)
       (effects (font (size 1.27 1.27)) hide)
     )
@@
       (effects (font (size 1.27 1.27)) (justify left))
     )
-    (property "Footprint" "" (at 332.232 344.17 90)
+    (property "Footprint" "Resistor_SMD:R_0805_2012Metric" (at 332.232 344.17 90)
       (effects (font (size 1.27 1.27)) hide)
     )
@@
       (effects (font (size 1.27 1.27)) (justify left))
     )
-    (property "Footprint" "SOT95P237X112-3N" (at 138.43 61.29 0)
+    (property "Footprint" "SamacSys_Parts:SOT95P237X112-3N" (at 138.43 61.29 0)
       (effects (font (size 1.27 1.27)) (justify left top) hide)
     )
@@
       (effects (font (size 1.27 1.27)) (justify left))
     )
-    (property "Footprint" "" (at 275.2852 306.07 0)
+    (property "Footprint" "Capacitor_SMD:C_0805_2012Metric" (at 275.2852 306.07 0)
       (effects (font (size 1.27 1.27)) hide)
     )
@@
       (effects (font (size 1.27 1.27)))
     )
-    (property "Footprint" "RJMG163118101NR" (at 372.11 240.36 0)
+    (property "Footprint" "SamacSys_Parts:RJMG163118101NR" (at 372.11 240.36 0)
       (effects (font (size 1.27 1.27)) (justify left top) hide)
     )
@@
       (effects (font (size 1.27 1.27)) (justify left))
     )
-    (property "Footprint" "" (at 285.4452 306.07 0)
+    (property "Footprint" "Capacitor_SMD:C_0805_2012Metric" (at 285.4452 306.07 0)
       (effects (font (size 1.27 1.27)) hide)
     )
@@
       (effects (font (size 1.27 1.27)) (justify left))
     )
-    (property "Footprint" "" (at 209.2452 368.3 0)
+    (property "Footprint" "Capacitor_SMD:C_0805_2012Metric" (at 209.2452 368.3 0)
       (effects (font (size 1.27 1.27)) hide)
     )
@@
       (effects (font (size 1.27 1.27)) (justify left))
     )
-    (property "Footprint" "" (at 334.9752 359.41 0)
+    (property "Footprint" "Capacitor_SMD:C_0805_2012Metric" (at 334.9752 359.41 0)
       (effects (font (size 1.27 1.27)) hide)
     )
@@
       (effects (font (size 1.27 1.27)) (justify left))
     )
-    (property "Footprint" "" (at 305.7652 306.07 0)
+    (property "Footprint" "Capacitor_SMD:C_0805_2012Metric" (at 305.7652 306.07 0)
       (effects (font (size 1.27 1.27)) hide)
     )
@@
       (effects (font (size 1.27 1.27)) (justify left))
     )
-    (property "Footprint" "" (at 409.702 342.9 90)
+    (property "Footprint" "Resistor_SMD:R_0805_2012Metric" (at 409.702 342.9 90)
       (effects (font (size 1.27 1.27)) hide)
     )
@@
       (effects (font (size 1.27 1.27)))
     )
-    (property "Footprint" "" (at 407.67 302.26 0)
+    (property "Footprint" "Inductor_SMD:L_0805_2012Metric" (at 407.67 302.26 0)
       (effects (font (size 1.27 1.27)) hide)
     )
@@
       (effects (font (size 1.27 1.27)) (justify left))
     )
-    (property "Footprint" "" (at 190.1952 368.3 0)
+    (property "Footprint" "Capacitor_SMD:C_0805_2012Metric" (at 190.1952 368.3 0)
       (effects (font (size 1.27 1.27)) hide)
     )
@@
       (effects (font (size 1.27 1.27)))
     )
-    (property "Footprint" "" (at 416.56 326.898 90)
+    (property "Footprint" "Resistor_SMD:R_0805_2012Metric" (at 416.56 326.898 90)
       (effects (font (size 1.27 1.27)) hide)
     )
@@
       (effects (font (size 1.27 1.27)))
     )
-    (property "Footprint" "" (at 347.98 329.8952 0)
+    (property "Footprint" "Capacitor_SMD:C_0805_2012Metric" (at 347.98 329.8952 0)
       (effects (font (size 1.27 1.27)) hide)
     )
@@
       (effects (font (size 1.27 1.27)) (justify left))
     )
-    (property "Footprint" "" (at 218.1352 313.69 0)
+    (property "Footprint" "Capacitor_SMD:C_0805_2012Metric" (at 218.1352 313.69 0)
       (effects (font (size 1.27 1.27)) hide)
     )
@@
       (effects (font (size 1.27 1.27)) (justify left))
     )
-    (property "Footprint" "" (at 322.072 307.34 90)
+    (property "Footprint" "Resistor_SMD:R_0805_2012Metric" (at 322.072 307.34 90)
       (effects (font (size 1.27 1.27)) hide)
     )
@@
       (effects (font (size 1.27 1.27)) (justify left))
     )
-    (property "Footprint" "" (at 244.8052 306.07 0)
+    (property "Footprint" "Capacitor_SMD:C_0805_2012Metric" (at 244.8052 306.07 0)
       (effects (font (size 1.27 1.27)) hide)
     )
@@
       (effects (font (size 1.27 1.27)))
     )
-    (property "Footprint" "" (at 271.78 374.9548 0)
+    (property "Footprint" "Capacitor_SMD:C_0805_2012Metric" (at 271.78 374.9548 0)
       (effects (font (size 1.27 1.27)) hide)
     )
@@
       (effects (font (size 1.27 1.27)))
     )
-    (property "Footprint" "" (at 341.63 330.708 90)
+    (property "Footprint" "Resistor_SMD:R_0805_2012Metric" (at 341.63 330.708 90)
       (effects (font (size 1.27 1.27)) hide)
     )
@@
       (effects (font (size 1.27 1.27)) (justify left))
     )
-    (property "Footprint" "SOT95P237X112-3N" (at 45.72 60.02 0)
+    (property "Footprint" "SamacSys_Parts:SOT95P237X112-3N" (at 45.72 60.02 0)
       (effects (font (size 1.27 1.27)) (justify left top) hide)
     )
@@
       (effects (font (size 1.27 1.27)) (justify left))
     )
-    (property "Footprint" "" (at 265.1252 306.07 0)
+    (property "Footprint" "Capacitor_SMD:C_0805_2012Metric" (at 265.1252 306.07 0)
       (effects (font (size 1.27 1.27)) hide)
     )
@@
       (effects (font (size 1.27 1.27)) (justify left))
     )
-    (property "Footprint" "" (at 323.342 344.17 90)
+    (property "Footprint" "Resistor_SMD:R_0805_2012Metric" (at 323.342 344.17 90)
       (effects (font (size 1.27 1.27)) hide)
     )
@@
       (effects (font (size 1.27 1.27)))
     )
-    (property "Footprint" "" (at 199.39 349.758 90)
+    (property "Footprint" "Resistor_SMD:R_0805_2012Metric" (at 199.39 349.758 90)
       (effects (font (size 1.27 1.27)) hide)
     )
@@
       (effects (font (size 1.27 1.27)) (justify left))
     )
-    (property "Footprint" "" (at 254.9652 306.07 0)
+    (property "Footprint" "Capacitor_SMD:C_0805_2012Metric" (at 254.9652 306.07 0)
       (effects (font (size 1.27 1.27)) hide)
     )
@@
       (effects (font (size 1.27 1.27)))
     )
-    (property "Footprint" "" (at 217.17 331.978 90)
+    (property "Footprint" "Resistor_SMD:R_0805_2012Metric" (at 217.17 331.978 90)
       (effects (font (size 1.27 1.27)) hide)
     )
@@
       (effects (font (size 1.27 1.27)) (justify left))
     )
-    (property "Footprint" "" (at 402.082 342.9 90)
+    (property "Footprint" "Resistor_SMD:R_0805_2012Metric" (at 402.082 342.9 90)
       (effects (font (size 1.27 1.27)) hide)
     )
@@
       (effects (font (size 1.27 1.27)))
     )
-    (property "Footprint" "" (at 341.63 324.358 90)
+    (property "Footprint" "Resistor_SMD:R_0805_2012Metric" (at 341.63 324.358 90)
       (effects (font (size 1.27 1.27)) hide)
     )
@@
       (effects (font (size 1.27 1.27)) (justify left))
     )
-    (property "Footprint" "" (at 329.692 307.34 90)
+    (property "Footprint" "Resistor_SMD:R_0805_2012Metric" (at 329.692 307.34 90)
       (effects (font (size 1.27 1.27)) hide)
     )
@@
       (effects (font (size 1.27 1.27)))
     )
-    (property "Footprint" "" (at 267.97 364.998 90)
+    (property "Footprint" "Resistor_SMD:R_0805_2012Metric" (at 267.97 364.998 90)
       (effects (font (size 1.27 1.27)) hide)
     )
@@
       (effects (font (size 1.27 1.27)))
     )
-    (property "Footprint" "" (at 355.6 334.3148 0)
-      (effects (font (size 1.27 1.27)) hide)
-    )
+    (property "Footprint" "Capacitor_SMD:C_0805_2012Metric" (at 355.6 334.3148 0)
+      (effects (font (size 1.27 1.27)) hide)
+    )

Commit message: Schematic update
* Remove USB-serial chip, use ESP32's USB support
* Add serial header and bootloader jumper in case that doesn't work
* Add drive current sensing
* ERC tidyup
* Add a few test points for good measure
Parts:
- removed C10: 10uF, Capacitor_SMD:C_0805_2012Metric, symbol Device:C_Small
- removed C11: 100nF, Capacitor_SMD:C_0805_2012Metric, symbol Device:C_Small
- removed Q1: UMH3N, SamacSys_Parts:SOT65P230X110-6N, symbol SamacSys_Parts:UMH3N
- removed U3: CH340C, Package_SO:SOIC-16_3.9x9.9mm_P1.27mm, symbol Interface_USB:CH340C
- added C4: 100nF, Capacitor_SMD:C_0805_2012Metric, symbol Device:C_Small
- added J7: FTDI, Connector_PinHeader_2.54mm:PinHeader_1x06_P2.54mm_Vertical, symbol Connector:Conn_01x06_Pin
- added JP1: Bootloader, TestPoint:TestPoint_2Pads_Pitch5.08mm_Drill1.3mm, symbol Jumper:Jumper_2_Open
- added R25: 0.015 R, Resistor_SMD:R_0805_2012Metric, symbol Device:R
- added R26: 10K, Resistor_SMD:R_0805_2012Metric, symbol Device:R
- added TP1: COIL_DRIVE_SENSE, TestPoint:TestPoint_Pad_D2.0mm, symbol Connector:TestPoint
- added TP2: COIL_DRIVE_IN, TestPoint:TestPoint_Pad_D2.0mm, symbol Connector:TestPoint
- added TP3: LED_IN, TestPoint:TestPoint_Pad_D2.0mm, symbol Connector:TestPoint
- added TP4: CS, TestPoint:TestPoint_Pad_D2.0mm, symbol Connector:TestPoint
- added TP5: SCLK, TestPoint:TestPoint_Pad_D2.0mm, symbol Connector:TestPoint
- added TP6: MISO, TestPoint:TestPoint_Pad_D2.0mm, symbol Connector:TestPoint
- added TP7: MOSI, Connector_PinHeader_2.54mm:PinHeader_1x06_P2.54mm_Vertical, symbol Connector:TestPoint
- added U4: NCS214, Package_TO_SOT_SMD:SOT-363_SC-70-6, symbol Amplifier_Current:NCS214
Connections:
- net +3V3: now also C4.1, R26.1, U4.3 (Vs)
- net COIL_DRIVE_IN: now also TP2.1
- net COIL_DRIVE_OUT: now also R25.2, U4.5 (-IN); no longer Q2.3 (D)
- net CS: now also TP4.1
- net ESP_RXD: now also J7.4 (Pin_4)
- net ESP_TXD: now also J7.5 (Pin_5)
- net GND: now also J6.S1, J6.S2, C4.2, J7.1 (Pin_1), JP1.1 (A), U4.1 (REF), U4.2 (GND)
- net IO0: now also JP1.2 (B), R26.2
- net LED_IN: now also TP3.1
- net MISO: now also TP6.1
- net MOSI: now also TP7.1
- net SCLK: now also TP5.1
- net USB_DN: now reaches U3.13 (GPIO19/U1RTS/ADC2_CH8/CLK_OUT2/USB_D-)
- net USB_DN: now also USB1.5 (DN2), USB1.7 (DN1)
- net USB_DP: now reaches U3.14 (GPIO20/U1CTS/ADC2_CH9/CLK_OUT1/USB_D+)
- net USB_DP: now also USB1.6 (DP1), USB1.8 (DP2)
- net COIL_DRIVE_SENSE: now reaches U3.15 (GPIO3/TOUCH3/ADC1_CH2)
- net COIL_DRIVE_SENSE: now also TP1.1, U4.6 (OUT)
- net at D3.2 (A): now also F1.2; no longer F1.1
- net USB_VBUS: now reaches USB1.11 (VBUS), USB1.2 (VBUS)
- net USB_VBUS: now also F1.1; no longer F1.2
- new net: Q2.3 (D), R25.1, U4.4 (+IN)
- no-connect marks 24 -> 20
Other:
- note removed: "USB UART"
- moved on the sheet: C4, C5, C8, D3, D4, F1, Q2, Q3, Q4, Q5, R12, R2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

Commit message: Rework schematic:
New 5V regulator design, use ESP32's native USB and add FTDI header,
misc other improvements
Parts:
- removed C2: 100uF, Capacitor_SMD:CP_Elec_10x10, symbol flipcontrol-rescue:CP-Device
- removed C5: 220uF, Capacitor_SMD:CP_Elec_10x10, symbol flipcontrol-rescue:CP-Device
- removed D1: D_Schottky, Diode_SMD:D_SMB, symbol Device:D_Schottky
- removed L1: 33uH, Inductor_SMD:L_12x12mm_H6mm, symbol flipcontrol-rescue:INDUCTOR-pspice
- removed R24: 4.7k, Resistor_SMD:R_0805_2012Metric, symbol Device:R
- removed U1: LM2596S-5, Package_TO_SOT_SMD:TO-263-5_TabPin3, symbol Regulator_Switching:LM2596S-5
- added C2: 10uF 2.8mΩ 35V, Capacitor_SMD:C_0805_2012Metric, symbol Device:C
- added C27: 47 pF, Capacitor_SMD:C_0805_2012Metric, symbol Device:C
- added C28: 47uF 3mΩ 16V, Capacitor_SMD:C_1210_3225Metric, symbol Device:C
- added C5: 100nF 30mΩ 50V, Capacitor_SMD:C_0805_2012Metric, symbol Device:C
- added C9: 100 nF 1mΩ 10V, Capacitor_SMD:C_0805_2012Metric, symbol Device:C_Small
- added D1: 5V, LED_SMD:LED_0805_2012Metric, symbol Device:LED
- added D5: 3V3, LED_SMD:LED_0805_2012Metric, symbol Device:LED
- added L1: IHLP4040DZER6R8M01, Inductor_SMD:L_Vishay_IHLP-4040, symbol Device:L
- added R27: 52.3k, Resistor_SMD:R_0805_2012Metric, symbol Device:R_Small
- added R28: 10k, Resistor_SMD:R_0805_2012Metric, symbol Device:R_Small
- added R29, R30: R_Small, Resistor_SMD:R_0805_2012Metric, symbol Device:R_Small
- added U1: TPS563300, Package_TO_SOT_SMD:SOT-583-8, symbol flipdot-controller:TPS563300
- JP1: footprint TestPoint:TestPoint_2Pads_Pitch5.08mm_Drill1.3mm -> digikey-footprints:Jumper_Tin_P5.32mm
- R20: value 12.4k -> 12.4k 1%
- TP7: footprint Connector_PinHeader_2.54mm:PinHeader_1x06_P2.54mm_Vertical -> TestPoint:TestPoint_Pad_D2.0mm
- U4: footprint Package_TO_SOT_SMD:SOT-363_SC-70-6 -> Package_TO_SOT_SMD:SOT-363_SC-70-6_Handsoldering
- USB1: footprint Type-C:HRO-TYPE-C-31-M-12 -> Connector_USB:USB_C_Receptacle_HRO_TYPE-C-31-M-12; symbol Type-C:HRO-TYPE-C-31-M-12 -> Connector:USB_C_Receptacle_USB2.0
Connections:
- net +3V3: now also R30.1
- net +5V: now also C27.1, C28.1, L1.2, R27.1, R29.1
- net GND: now also C14.1, C15.1, USB1.A1 (GND), USB1.A12 (GND), USB1.B1 (GND), USB1.B12 (GND), USB1.S1 (SHIELD), C2.2, C28.2, C5.2, D1.1 (K), D5.1 (K), R28.2, U1.4 (GND); no longer C14.2, C15.2, USB1.1 (GND), USB1.12 (GND), USB1.13 (SHIELD)
- net USB_DN: now also USB1.A7 (D-), USB1.B7 (D-); no longer USB1.5 (DN2), USB1.7 (DN1)
- net USB_DP: now also USB1.A6 (D+), USB1.B6 (D+); no longer USB1.6 (DP1), USB1.8 (DP2)
- net USB_VBUS: now also USB1.A4 (VBUS), USB1.A9 (VBUS), USB1.B4 (VBUS), USB1.B9 (VBUS); no longer USB1.11 (VBUS), USB1.2 (VBUS)
- net at U5.20 (TOCAP): now also C15.2; no longer C15.1
- net at U5.22 (1V2O): now also C14.2; no longer C14.1
- net at R4.2: now also USB1.B5 (CC2); no longer USB1.10 (CC2)
- net at R3.2: now also USB1.A5 (CC1); no longer USB1.4 (CC1)
- net +24V renamed +18V
- net +18V: now also C2.1, C5.1, U1.3 (VIN)
- new net: C27.2, R27.2, R28.1, U1.8 (VFB)
- new net: D5.2 (A), R30.2
- new net: D1.2 (A), R29.2
- new net: C9.1, L1.1, U1.5 (SW)
- new net: C9.2, U1.6 (VBST)
- no-connect marks 20 -> 22
Other:
- note added: "18V Power Budget: 5 V supply (13 W output, 1.4 W regulator loss): 1.25A Pixel drive current: 2A (?) Total: 3.25 A (58.5 W)"
- note added: "3.3V Power budget: ESP32-S3: 500 mA W5500: 132 mA NCS214: 10 mA Total: 0.642 A (2.1 W) AMS1117 rating: 1 A"
- note added: "5V Power Budget: 3.3 V supply (2.2W draw, 1.1W regulator loss): 1500 mA Panels x3: 1000 mA (estimate) Total: 2.5 A (12.5 W) Regulator design rating: 3A"
- moved on the sheet: C10, C11, C12, C13, C14, C15, C16, C17, C18, C19, C20, C21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
