File: pcb/flipcontrol.kicad_sch (KiCad schematic)
At the start: 96 parts, among them J1 PJ-202A, J2 DOT_BOARD_1, J3 DOT_BOARD_2, J4 LED_STRIP, J5 DOT_BOARD_3, J6 RJMG163118101NR, J7 FTDI, Q2 Si2347DS-T1-GE3, Q3 MMBT3904, Q4 Si2347DS-T1-GE3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

Commit message: Schematic updates to improve component values
Parts:
- C2: value 10uF 2.8mΩ 35V -> 10uF; ESR (none) -> 2.8mΩ; Voltage (none) -> 35V
- C22: value 10uF/16V -> 10uF; Rating (none) -> 16V
- C23: value 10uF/16v -> 10uF; Voltage (none) -> 16V
- C27: value 47 pF -> 47pF
- C28: value 47uF 3mΩ 16V -> 47uF; ESR (none) -> 3mΩ; Voltage (none) -> 16V
- C5: value 100nF 30mΩ 50V -> 100nF; ESR (none) -> 30mΩ; Voltage (none) -> 50V
- C9: value 100 nF 1mΩ 10V -> 100nF; ESR (none) -> 1mΩ; Voltage (none) -> 10V
- L1: value IHLP4040DZER6R8M01 -> 6.8uH; Part (none) -> IHLP4040DZER6R8M01
- L2: value HH-1M1608-121JT -> ~; symbol Device:L -> Device:FerriteBead_Small
- R20: value 12.4k 1% -> 12.4k; Tolerance (none) -> 1%
- R29: value R_Small -> 145R
- R30: value R_Small -> 60R
Changed lines of the file:
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@@
     (stroke (width 0) (type default))
   )
-  (wire (pts (xy 273.685 279.4) (xy 283.845 279.4))
+  (wire (pts (xy 273.685 279.4) (xy 285.115 279.4))
     (stroke (width 0) (type default))
   )
@@
     (stroke (width 0) (type default))
   )
-  (wire (pts (xy 291.465 279.4) (xy 300.355 279.4))
+  (wire (pts (xy 290.195 279.4) (xy 300.355 279.4))
     (stroke (width 0) (type default))
   )
@@
       (effects (font (size 1.27 1.27)) (justify left))
     )
-    (property "Value" "47 pF" (at 110.49 266.065 0)
+    (property "Value" "47pF" (at 110.49 266.065 0)
       (effects (font (size 1.27 1.27)) (justify left))
     )
@@
   (symbol (lib_id "Device:D_Schottky") (at 121.92 222.885 180) (unit 1)
     (in_bom yes) (on_board yes) (dnp no)
-    (property "Reference" "D3" (at 123.0884 224.917 90)
+    (property "Reference" "D3" (at 121.92 229.235 0)
       (effects (font (size 1.27 1.27)) (justify left))
     )
-    (property "Value" "D" (at 120.777 224.917 90)
+    (property "Value" "D" (at 120.65 226.06 0)
       (effects (font (size 1.27 1.27)) (justify left))
     )
@@
   )
   (symbol (lib_id "Device:C") (at 137.795 264.16 0) (unit 1)
-    (in_bom yes) (on_board yes) (dnp no) (fields_autoplaced)
+    (in_bom yes) (on_board yes) (dnp no)
     (property "Reference" "C28" (at 140.97 263.525 0)
       (effects (font (size 1.27 1.27)) (justify left))
     )
-    (property "Value" "47uF 3mΩ 16V" (at 140.97 266.065 0)
+    (property "Value" "47uF" (at 140.97 266.065 0)
       (effects (font (size 1.27 1.27)) (justify left))
     )
@@
       (effects (font (size 1.27 1.27)) hide)
     )
+    (property "ESR" "3mΩ" (at 140.97 269.875 0)
+      (effects (font (size 1.27 1.27)) (justify left))
+    )
+    (property "Voltage" "16V" (at 140.97 267.97 0)
+      (effects (font (size 1.27 1.27)) (justify left))
+    )
     (pin "1")
     (pin "2")
@@
   )
   (symbol (lib_id "Device:C_Polarized") (at 390.525 278.13 0) (unit 1)
-    (in_bom yes) (on_board yes) (dnp no) (fields_autoplaced)
-    (property "Reference" "C22" (at 393.446 276.5973 0)
+    (in_bom yes) (on_board yes) (dnp no)
+    (property "Reference" "C22" (at 393.7 276.86 0)
       (effects (font (size 1.27 1.27)) (justify left))
     )
-    (property "Value" "10uF/16V" (at 393.446 278.5183 0)
+    (property "Value" "10uF" (at 393.7 278.765 0)
       (effects (font (size 1.27 1.27)) (justify left))
     )
@@
       (effects (font (size 1.27 1.27)) hide)
     )
+    (property "Rating" "16V" (at 395.605 280.67 0)
+      (effects (font (size 1.27 1.27)))
+    )
     (pin "1")
     (pin "2")
@@
     )
   )
-  (symbol (lib_id "Device:L") (at 287.655 279.4 90) (unit 1)
-    (in_bom yes) (on_board yes) (dnp no) (fields_autoplaced)
-    (property "Reference" "L2" (at 287.655 275.8847 90)
+  (symbol (lib_id "Device:FerriteBead_Small") (at 287.655 279.4 90) (unit 1)
+    (in_bom yes) (on_board yes) (dnp no)
+    (property "Reference" "L2" (at 287.655 275.59 90)
       (effects (font (size 1.27 1.27)))
     )
-    (property "Value" "HH-1M1608-121JT" (at 287.655 277.8057 90)
+    (property "Value" "~" (at 287.655 277.495 90)
       (effects (font (size 1.27 1.27)))
     )
-    (property "Footprint" "Inductor_SMD:L_0805_2012Metric" (at 287.655 279.4 0)
+    (property "Footprint" "Inductor_SMD:L_0805_2012Metric" (at 287.655 281.178 90)
       (effects (font (size 1.27 1.27)) hide)
     )
@@
   )
   (symbol (lib_id "power:+3V3") (at 162.56 257.175 0) (unit 1)
-    (in_bom yes) (on_board yes) (dnp no) (fields_autoplaced)
+    (in_bom yes) (on_board yes) (dnp no)
     (property "Reference" "#PWR060" (at 162.56 260.985 0)
       (effects (font (size 1.27 1.27)) hide)
     )
-    (property "Value" "+3V3" (at 162.56 254 0)
+    (property "Value" "+3V3" (at 161.925 253.365 0)
       (effects (font (size 1.27 1.27)))
     )
@@
   )
   (symbol (lib_id "Device:C_Polarized") (at 250.825 280.67 0) (unit 1)
-    (in_bom yes) (on_board yes) (dnp no) (fields_autoplaced)
-    (property "Reference" "C23" (at 253.746 279.1373 0)
+    (in_bom yes) (on_board yes) (dnp no)
+    (property "Reference" "C23" (at 254 279.4 0)
       (effects (font (size 1.27 1.27)) (justify left))
     )
-    (property "Value" "10uF/16v" (at 253.746 281.0583 0)
+    (property "Value" "10uF" (at 254 281.305 0)
       (effects (font (size 1.27 1.27)) (justify left))
     )
@@
     )
     (property "Datasheet" "~" (at 250.825 280.67 0)
-      (effects (font (size 1.27 1.27)) hide)
+      (effects (font (size 1.27 1.27)) (justify left))
+    )
+    (property "Voltage" "16V" (at 254 283.21 0)
+      (effects (font (size 1.27 1.27)) (justify left))
     )
     (pin "1")
@@
       (effects (font (size 1.27 1.27)))
     )
-    (property "Value" "100 nF 1mΩ 10V" (at 90.17 264.795 90)
+    (property "Value" "100nF" (at 85.725 264.795 90)
       (effects (font (size 1.27 1.27)))
     )
@@
       (effects (font (size 1.27 1.27)) hide)
     )
+    (property "ESR" "1mΩ" (at 91.44 264.795 90)
+      (effects (font (size 1.27 1.27)))
+    )
+    (property "Voltage" "10V" (at 96.52 264.795 90)
+      (effects (font (size 1.27 1.27)))
+    )
     (pin "1")
     (pin "2")
@@
       (effects (font (size 1.27 1.27)))
     )
-    (property "Value" "R_Small" (at 171.45 247.65 90)
+    (property "Value" "145R" (at 171.45 247.65 90)
       (effects (font (size 1.27 1.27)))
     )
@@
   (symbol (lib_id "Device:L") (at 99.06 259.08 90) (unit 1)
     (in_bom yes) (on_board yes) (dnp no)
-    (property "Reference" "L1" (at 99.06 254 90)
+    (property "Reference" "L1" (at 99.06 251.46 90)
       (effects (font (size 1.27 1.27)))
     )
-    (property "Value" "IHLP4040DZER6R8M01" (at 99.06 256.54 90)
+    (property "Value" "6.8uH" (at 99.06 254 90)
       (effects (font (size 1.27 1.27)))
     )
@@
       (effects (font (size 1.27 1.27)) hide)
     )
+    (property "Part" "IHLP4040DZER6R8M01" (at 99.06 256.54 90)
+      (effects (font (size 1.27 1.27)))
+    )
     (pin "1")
     (pin "2")
@@
       (effects (font (size 1.27 1.27)) hide)
     )
-    (property "Value" "+5V" (at 135.2042 223.266 90)
+    (property "Value" "+5V" (at 135.89 222.885 90)
       (effects (font (size 1.27 1.27)))
     )
@@
       (effects (font (size 1.27 1.27)))
     )
-    (property "Value" "R_Small" (at 171.45 256.54 90)
+    (property "Value" "60R" (at 171.45 256.54 90)
       (effects (font (size 1.27 1.27)))
     )
@@
   (symbol (lib_id "Device:R") (at 275.59 363.22 90) (unit 1)
     (in_bom yes) (on_board yes) (dnp no)
-    (property "Reference" "R20" (at 275.59 358.14 90)
+    (property "Reference" "R20" (at 275.59 355.6 90)
       (effects (font (size 1.27 1.27)))
     )
-    (property "Value" "12.4k 1%" (at 275.59 360.68 90)
+    (property "Value" "12.4k" (at 275.59 358.14 90)
       (effects (font (size 1.27 1.27)))
     )
@@
       (effects (font (size 1.27 1.27)) hide)
     )
+    (property "Tolerance" "1%" (at 275.59 360.045 90)
+      (effects (font (size 1.27 1.27)))
+    )
     (pin "1")
     (pin "2")
@@
       (effects (font (size 1.27 1.27)) (justify left))
     )
-    (property "Value" "10uF 2.8mΩ 35V" (at 29.845 264.795 0)
+    (property "Value" "10uF" (at 29.845 264.16 0)
       (effects (font (size 1.27 1.27)) (justify left))
     )
@@
       (effects (font (size 1.27 1.27)) hide)
     )
+    (property "ESR" "2.8mΩ" (at 29.845 266.065 0)
+      (effects (font (size 1.27 1.27)) (justify left))
+    )
+    (property "Voltage" "35V" (at 29.845 267.97 0)
+      (effects (font (size 1.27 1.27)) (justify left))
+    )
     (pin "1")
     (pin "2")
@@
       (effects (font (size 1.27 1.27)) (justify left))
     )
-    (property "Value" "100nF 30mΩ 50V" (at 41.275 266.065 0)
+    (property "Value" "100nF" (at 43.815 264.16 0)
       (effects (font (size 1.27 1.27)) (justify left))
     )
@@
       (effects (font (size 1.27 1.27)) hide)
     )
+    (property "ESR" "30mΩ" (at 43.815 266.065 0)
+      (effects (font (size 1.27 1.27)) (justify left))
+    )
+    (property "Voltage" "50V" (at 43.815 267.97 0)
+      (effects (font (size 1.27 1.27)) (justify left))
+    )
     (pin "1")
