File: pcb/flipcontrol.kicad_sch (KiCad schematic)
At the start: 92 parts, among them J1 PJ-202A, J2 DOT_BOARD_1, J3 DOT_BOARD_2, J4 LED_STRIP, J5 DOT_BOARD_3, J6 RJMG163118101NR, J7 FTDI, Q2 Si2347DS-T1-GE3, Q3 MMBT3904, Q4 Si2347DS-T1-GE3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

Commit message: Rev4: Make more parts JLCPCB assembly service compatible
Parts:
- C8: LCSC C440198 -> C49678
- D2: LCSC C64898 -> C84256
- D3: LCSC C84256 -> C64898
- L2: value ~ -> 120Ohms@100MHz; LCSC (none) -> C88990
- L3: footprint Inductor_SMD:L_Vishay_IHLP-6767 -> Inductor_SMD:L_Sunlord_MWSA1206S-470; LCSC C6577597 -> C408531
- R29: LCSC (none) -> C17540
- U4: LCSC (none) -> C603836
- Y1: LCSC (none) -> C596913
