File: pcb/flipcontrol.kicad_pcb (KiCad board)
At the start: 4 copper layers, 133.3 x 61.6 mm, 96 parts, among them J1 PJ-202A, J2 DOT_BOARD_1, J3 DOT_BOARD_2, J4 LED_STRIP, J5 DOT_BOARD_3, J6 RJMG163118101NR, J7 FTDI, Q2 Si2347DS-T1-GE3, Q3 MMBT3904, Q4 Si2347DS-T1-GE3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

Commit message: JLCPB parts update
Parts:
- L2: value HH-1M1608-121JT -> 120Ohms@100MHz
- R29: value R_Small -> 145R
- R30: value R_Small -> 60R
Other:
- board text added: "Revision 5.0"
- board text removed: "Revision 1.0"
